File: PROGBK1/cartridge_edge.kicad_sch (KiCad schematic)
At the start: 3 parts, among them CN2 PROG Board

Commit message: Updated schematics and PCB layout
Parts:
- C1, C2: footprint (none) -> Capacitor_SMD:C_0805_2012Metric_Pad1.18x1.45mm_HandSolder
- CN2: footprint (none) -> Neo Geo:Connector_PCBEdge_Cartridge_2x60_P2.54mm_Edge
Connections:
- net 5V: now also CN2.A30, CN2.A31, CN2.B30, CN2.B31; no longer CN2.a30, CN2.a31, CN2.b30, CN2.b31
- net 68KCLKB: now also CN2.B24; no longer CN2.b24
- net A1: now also CN2.B5; no longer CN2.b5
- net A10: now also CN2.B14; no longer CN2.b14
- net A11: now also CN2.B15; no longer CN2.b15
- net A12: now also CN2.B16; no longer CN2.b16
- net A13: now also CN2.B17; no longer CN2.b17
- net A14: now also CN2.B18; no longer CN2.b18
- net A15: now also CN2.B19; no longer CN2.b19
- net A16: now also CN2.B20; no longer CN2.b20
- net A17: now also CN2.B21; no longer CN2.b21
- net A18: now also CN2.B22; no longer CN2.b22
- net A19: now also CN2.B23; no longer CN2.b23
- net A2: now also CN2.B6; no longer CN2.b6
- net A3: now also CN2.B7; no longer CN2.b7
- net A4: now also CN2.B8; no longer CN2.b8
- net A5: now also CN2.B9; no longer CN2.b9
- net A6: now also CN2.B10; no longer CN2.b10
- net A7: now also CN2.B11; no longer CN2.b11
- net A8: now also CN2.B12; no longer CN2.b12
- net A9: now also CN2.B13; no longer CN2.b13
- net D0: now also CN2.A5; no longer CN2.a5
- net D1: now also CN2.A6; no longer CN2.a6
- net D10: now also CN2.A15; no longer CN2.a15
- net D11: now also CN2.A16; no longer CN2.a16
- net D12: now also CN2.A17; no longer CN2.a17
- net D13: now also CN2.A18; no longer CN2.a18
- net D14: now also CN2.A19; no longer CN2.a19
- net D15: now also CN2.A20; no longer CN2.a20
- net D2: now also CN2.A7; no longer CN2.a7
- net D3: now also CN2.A8; no longer CN2.a8
- net D4: now also CN2.A9; no longer CN2.a9
- net D5: now also CN2.A10; no longer CN2.a10
- net D6: now also CN2.A11; no longer CN2.a11
- net D7: now also CN2.A12; no longer CN2.a12
- net D8: now also CN2.A13; no longer CN2.a13
- net D9: now also CN2.A14; no longer CN2.a14
- net GND: now also CN2.A1, CN2.A2, CN2.A3, CN2.A4, CN2.A57, CN2.A58, CN2.A59, CN2.A60, CN2.B1, CN2.B2, CN2.B3, CN2.B4, CN2.B57, CN2.B58, CN2.B59, CN2.B60; no longer CN2.a1, CN2.a2, CN2.a3, CN2.a4, CN2.a57, CN2.a58, CN2.a59, CN2.a60, CN2.b1, CN2.b2, CN2.b3, CN2.b4, CN2.b57, CN2.b58, CN2.b59, CN2.b60
- net PDTACK: now also CN2.B28; no longer CN2.b28
- net PORTADRS: now also CN2.A33; no longer CN2.a33
- net PORTOEL: now also CN2.A26; no longer CN2.a26
- net PORTOEU: now also CN2.A25; no longer CN2.a25
- net PWAIT0: now also CN2.B26; no longer CN2.b26
- net PWAIT1: now also CN2.B27; no longer CN2.b27
- net RESET: now also CN2.B35; no longer CN2.b35
- net ROMWAIT: now also CN2.B25; no longer CN2.b25
- net SDPA10: now also CN2.A45; no longer CN2.a45
- net SDPA11: now also CN2.A46; no longer CN2.a46
- net SDPA8: now also CN2.A43; no longer CN2.a43
- net SDPA9: now also CN2.A44; no longer CN2.a44
- net SDPAD0: now also CN2.B41; no longer CN2.b41
- net SDPAD1: now also CN2.B42; no longer CN2.b42
- net SDPAD2: now also CN2.B43; no longer CN2.b43
- net SDPAD3: now also CN2.B44; no longer CN2.b44
- net SDPAD4: now also CN2.B45; no longer CN2.b45
- net SDPAD5: now also CN2.B46; no longer CN2.b46
- net SDPAD6: now also CN2.B47; no longer CN2.b47
- net SDPAD7: now also CN2.B48; no longer CN2.b48
- net SDPMPX: now also CN2.A47; no longer CN2.a47
- net SDPOE: now also CN2.A48; no longer CN2.a48
- net SDRA20: now also CN2.A51; no longer CN2.a51
- net SDRA21: now also CN2.A52; no longer CN2.a52
- net SDRA22: now also CN2.A53; no longer CN2.a53
- net SDRA23: now also CN2.A54; no longer CN2.a54
- net SDRA8: now also CN2.A50; no longer CN2.a50
- net SDRA9: now also CN2.A49; no longer CN2.a49
- net SDRAD0: now also CN2.B49; no longer CN2.b49
- net SDRAD1: now also CN2.B50; no longer CN2.b50
- net SDRAD2: now also CN2.B51; no longer CN2.b51
- net SDRAD3: now also CN2.B52; no longer CN2.b52
- net SDRAD4: now also CN2.B53; no longer CN2.b53
- net SDRAD5: now also CN2.B54; no longer CN2.b54
- net SDRAD6: now also CN2.B55; no longer CN2.b55
- net SDRAD7: now also CN2.B56; no longer CN2.b56
- net SDRMPX: now also CN2.A55; no longer CN2.a55
- net SDROE: now also CN2.A56; no longer CN2.a56
- net ~{PORTWEL}: now also CN2.A28; no longer CN2.a28
- net ~{ROMOE}: now also CN2.B33; no longer CN2.b33
